File: nucleo-144.kicad_sch (KiCad schematic)
At the start: 3 parts, among them U4 NUCLEO144-H743ZI

Commit message: - Removed I2C lines - Added mission resistor between buffer and transistor gate - Removed wetting current & high range enable - Added ILI9341 TFT LCD - Removed OLED - Upped current gain to ~100
Parts:
- removed R25, R26: 2k2, PCM_Resistor_SMD_AKL:R_0603_1608Metric, symbol PCM_Resistor_AKL:R_0603
Connections:
- net TMC2209_VREF: now reaches U4.CN7_12 (PA6)
- net TMC2209_MS1: now reaches U4.CN9_13 (РВ2)
- net TMC2209_MS2: now reaches U4.CN9_14 (PE2)
- net TMC2209_CLK: now reaches U4.CN9_15 (РЕ9)
- net TMC2209_DIR: now reaches U4.CN9_17 (PF2)
- net TMC2209_STEP: now reaches U4.CN9_18 (РЕ5)
- net ILI9341_SPI_MISO: now reaches U4.CN9_24 (PF8)
- net ILI9341_SPI_CS: now reaches U4.CN9_25 (PD0)
- net ILI9341_SPI_SCK: now reaches U4.CN9_26 (PF7)
- net ILI9341_RESET: now reaches U4.CN9_27 (PD1)
- net ILI9341_SPI_MOSI: now reaches U4.CN9_28 (PF9)
- net ILI9341_SPI_DC: now reaches U4.CN9_30 (PG1)
- net TMC2209_RX: now reaches U4.CN9_4 (PD6)
- net TMC2209_DIAG: now reaches U4.CN9_5 (РСЗ)
- net TMC2209_TX: now reaches U4.CN9_6 (PD5)
- net TMC2209_EN: now reaches U4.CN9_8 (PD4)
- net EN_WETTING_CURRENT: no longer names the net of U4.CN10_21 (PD12)
- net E_HIGH_I_RANGE: no longer names the net of U4.CN10_2 (PG12)
- net I2C_SCK: no longer names the net of U4.CN9_19 (PF1)
- net I2C_SDA: no longer names the net of U4.CN9_21 (PF0)
