File: power.kicad_sch (KiCad schematic)
At the start: 17 parts, among them U5 MCP1501-30xCH

Commit message: - Removed I2C lines - Added mission resistor between buffer and transistor gate - Removed wetting current & high range enable - Added ILI9341 TFT LCD - Removed OLED - Upped current gain to ~100
Parts:
- removed LED2: LED_0805_Red, PCM_LED_SMD_AKL:LED_0805_2012Metric, symbol PCM_LED_AKL:LED_0805_Red
- removed R27: 4k7, PCM_Resistor_SMD_AKL:R_0603_1608Metric, symbol PCM_Resistor_AKL:R_0603
- removed TP3, TP4, TP5, TP6, TP7, TP8: GND, TestPoint:TestPoint_THTPad_D1.0mm_Drill0.5mm, symbol Connector:TestPoint
