File: user_interface.kicad_sch (KiCad schematic)
At the start: 19 parts, among them SW1 VAL?, SW2 VAL?, SW3 RotaryEncoder_Switch_MP

Commit message: - Removed I2C lines - Added mission resistor between buffer and transistor gate - Removed wetting current & high range enable - Added ILI9341 TFT LCD - Removed OLED - Upped current gain to ~100
Parts:
- removed C22: 100n, PCM_Capacitor_SMD_AKL:C_0603_1608Metric, symbol PCM_Capacitor_AKL:C_0603
- removed U6: ~, athanniss-lcd:SSD1306-0.91-OLED-4pin-128x32_no-header-offset, symbol PrivateLib:SSD1306-128x32-0.91
- added C22: 100 uF, PCM_Capacitor_SMD_AKL:C_Elec_6.3x7.7, symbol PCM_Capacitor_AKL:C_Bipolar_SMD_D6.3mm_H5.8mm
- added J4: Conn_01x04, Connector_JST:JST_PH_S4B-PH-K_1x04_P2.00mm_Horizontal, symbol Connector_Generic:Conn_01x04
- added U6: CR2013-MI2120, Display:CR2013-MI2120, symbol Driver_Display:CR2013-MI2120
- added U7: ~, athaniss-device:BTT-TMC2209-V1.3_RAISED, symbol athanniss-lib:BTT-TMC2209-V1.3
- renumbered R28 to R24, R29 to R25, R30 to R26, R31 to R27, R32 to R28, R33 to R29, R34 to R30, R35 to R31
Connections:
- net +3V3: now also U6.1 (VCC), U6.8 (LED), U7.10 (VDD)
- net GND: now also U6.2 (GND), U7.9 (GND)
- new net: J4.4 (Pin_4), U7.11 (B2)
- new net: J4.3 (Pin_3), U7.12 (B1)
- new net: J4.2 (Pin_2), U7.13 (A1)
- new net: J4.1 (Pin_1), U7.14 (A2)
- new net +12V: C22.1, U7.16 (VMOT)
- new net GNDPWR: C22.2, U7.15 (GND)
- new net ILI9341_RESET: U6.4 (RESET)
- new net ILI9341_SPI_CS: U6.3 (~{CS})
- new net ILI9341_SPI_DC: U6.5 (D/~{C})
- new net ILI9341_SPI_MISO: U6.9 (MISO)
- new net ILI9341_SPI_MOSI: U6.6 (MOSI)
- new net ILI9341_SPI_SCK: U6.7 (SCK)
- new net TMC2209_CLK: U7.6 (CLK)
- new net TMC2209_DIAG: U7.17 (DIAG)
- new net TMC2209_DIR: U7.8 (DIR)
- new net TMC2209_EN: U7.1 (EN)
- new net TMC2209_MS1: U7.2 (MS1)
- new net TMC2209_MS2: U7.3 (MS2)
- new net TMC2209_RX: U7.4 (Rx)
- new net TMC2209_STEP: U7.7 (STEP)
- new net TMC2209_TX: U7.5 (Tx)
- new net TMC2209_VREF: U7.18 (VREF)
Other:
- moved on the sheet: C19, C20, C21, R24, R26, R28, R30, R31, SW1, SW2, SW3
