File: output_analog.kicad_sch (KiCad schematic)
At the start: 38 parts, among them Q1 DMTH10H009LPSQ-13, U1 TSV732IS, U2 74LVC1G17, U3 TSV732IS

Commit message: Cleaned up unecessary HMI, optimized sheets.
Other:
- note added: "Voltage Measurement"
- title: (none) -> Procyon [Capstone]
- moved on the sheet: C1, C10, C11, C2, C3, C4, C5, C6, C7, C8, C9, D1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

Commit message: Added HS current sense to analog chain. Refactored schematics. Added snubber to the n-fet. Moved some stuff to DNP for clarity.
Parts:
- removed LED1: LED_0805_Red, PCM_LED_SMD_AKL:LED_0805_2012Metric, symbol PCM_LED_AKL:LED_0805_Red
- removed R7: 4k7, PCM_Resistor_SMD_AKL:R_0603_1608Metric, symbol PCM_Resistor_AKL:R_0603
- added C19, C20: 100n, PCM_Capacitor_SMD_AKL:C_0603_1608Metric, symbol PCM_Capacitor_AKL:C_0603
- added C21: 0, PCM_Capacitor_SMD_AKL:C_0603_1608Metric, symbol PCM_Capacitor_AKL:C_0603
- added R21: 0.015R, PCM_Resistor_SMD_AKL:R_1206_3216Metric, symbol athanniss-lib:MFSA1206R0150FCM
- added R22: 220R, PCM_Resistor_SMD_AKL:R_0603_1608Metric, symbol PCM_Resistor_AKL:R_0603
- added R7: R, Resistor_SMD:R_0805_2012Metric, symbol Device:R
- added TP1: TestPoint, Connector_PinHeader_2.00mm:PinHeader_1x01_P2.00mm_Vertical, symbol Connector:TestPoint
- added U6: INA240A2D, Package_SO:SOIC-8_3.9x4.9mm_P1.27mm, symbol Amplifier_Current:INA240A2D
- C1, C5: value 100n -> 10n
- C6, R15: now not fitted
Connections:
- net +12V: now also R21.1, U6.8 (+)
- net +5VA: now also C19.1, U6.6 (V+)
- net GND: now also C19.2, C20.2, U6.2 (GND), U6.3 (REF2), U6.4 (GND), U6.7 (REF1)
- net at Q1.S, R14.1, R9.1: now also C21.2
- net I_MEAS renamed MEAS_ILS
- net LS1_RETURN renamed COIL_IN
- net COIL_IN: now also R7.1
- net V24_MEAS renamed MEAS_VBUS
- net V_NFET_MEAS renamed MEAS_VFET
- new net: C21.1, R7.2
- new net: R22.1, U6.5
- new net COIL_OUT: R21.2, U6.1 (-)
- new net MEAS_IHS: C20.1, R22.2
Other:
- note added: "HS Current Sense"
- note added: "LS Current Sense"
- note added: "PWM Driver"
- moved on the sheet: C1, C10, C11, C2, C3, C4, C5, C7, C8, C9, D1, NT1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

Commit message: Refactored Nucleo sheet. Added back my library. Started minor work on the PCB.
Parts:
- added TP2, TP3, TP4, TP5, TP6, TP7: TestPoint, Connector_PinHeader_2.00mm:PinHeader_1x01_P2.00mm_Vertical, symbol Connector:TestPoint
Connections:
- net MEAS_IHS: now also TP2.1
- net MEAS_ILS: now also TP3.1
- net MEAS_VBUS: now also TP5.1
- net MEAS_VFET: now also TP4.1
- net at C5.1, R12.2, U1.5 (+): now also TP7.1
- net at TP1.1: now also Q1.G, R6.2, R8.2
- net at C1.1, R3.2, U1.3 (+): now also TP6.1
Other:
- moved on the sheet: TP1

Commit message: Finalized V1.1. Refactor schematics (PCB is ripped up) for HS measurement. Kept LS custom chain for reference.
Parts:
- added TP15: TestPoint, Connector_PinHeader_2.00mm:PinHeader_1x01_P2.00mm_Vertical, symbol Connector:TestPoint
- C21: value 0 -> (none)
- R6: value 1k -> 100R
- R7: value R -> (none)
Connections:
- net +12V: now also TP15.1
Changed lines of the file:
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@@
 	(title_block
 		(title "Procyon [Capstone]")
-		(rev "V1.1.x")
+		(date "2026-09-22")
+		(rev "V1.1.0")
+		(comment 1 "Not intended for production. Keeps custom I_LS chain for future reference.")
 	)
 	(rectangle
@@
 		)
 	)
+	(text_box "RC snubber to dampen potential ringing:\n+---------+-------------------+\n| C21     | R7 values to try  |\n+---------+-------------------+\n| 470 pF  | 10R, 22R, 33R     |\n| 1 nF    | 10R, 22R, 33R     |\n| 2.2 nF  | 10R, 15R, 22R     |\n| 4.7 nF  | 4R7, 10R, 15R     |\n+---------+-------------------+\n\nSuggested starting point:\nC21 = 1 nF - C0G/100V\nR7  = 22R - Size 0805"
+		(exclude_from_sim no)
+		(at 161.29 144.78 0)
+		(size 40.64 29.2948)
+		(margins 0.9525 0.9525 0.9525 0.9525)
+		(stroke
+			(width 0)
+			(type solid)
+		)
+		(fill
+			(type none)
+		)
+		(effects
+			(font
+				(face "Consolas")
+				(size 1.27 1.27)
+			)
+			(justify left top)
+		)
+	)
 	(text_box "Vout_max = Rsense * Imax * Gain\n\n	- A2 gain = 50\n	- A3 gain = 100\n\nRsense = 0.015\nImax = 2\n\nA2 Vout_max = 1,5V\nA3 Vout_max = 3,0V\n"
 		(exclude_from_sim no)
@@
 	)
 	(junction
+		(at 140.97 76.2)
+		(diameter 0)
+		(color 0 0 0 0)
+	)
+	(junction
 		(at 220.98 215.9)
 		(diameter 0)
@@
 	(wire
 		(pts
-			(xy 140.97 69.85) (xy 140.97 88.9)
+			(xy 140.97 69.85) (xy 140.97 76.2)
 		)
 		(stroke
@@
 	(wire
 		(pts
+			(xy 140.97 76.2) (xy 140.97 88.9)
+		)
+		(stroke
+			(width 0)
+			(type default)
+		)
+	)
+	(wire
+		(pts
 			(xy 312.42 157.48) (xy 312.42 158.75)
 		)
@@
 	(wire
 		(pts
+			(xy 128.27 71.12) (xy 128.27 76.2)
+		)
+		(stroke
+			(width 0)
+			(type default)
+		)
+	)
+	(wire
+		(pts
 			(xy 274.32 213.36) (xy 279.4 213.36)
 		)
@@
 	(wire
 		(pts
+			(xy 128.27 76.2) (xy 140.97 76.2)
+		)
+		(stroke
+			(width 0)
+			(type default)
+		)
+	)
+	(wire
+		(pts
 			(xy 294.64 135.89) (xy 294.64 138.43)
 		)
@@
 			)
 		)
-		(property "Value" "0"
+		(property "Value" ""
 			(at 154.178 166.37 0)
 			(hide yes)
@@
 			)
 		)
-		(property "Value" "R"
+		(property "Value" ""
 			(at 153.67 154.9399 0)
 			(hide yes)
@@
 	)
 	(symbol
+		(lib_id "Connector:TestPoint")
+		(at 128.27 71.12 0)
+		(unit 1)
+		(body_style 1)
+		(exclude_from_sim no)
+		(in_bom yes)
+		(on_board yes)
+		(in_pos_files yes)
+		(dnp no)
+		(property "Reference" "TP15"
+			(at 126.746 65.786 0)
+			(show_name no)
+			(do_not_autoplace no)
+			(effects
+				(font
+					(size 1.27 1.27)
+				)
+				(justify left)
+			)
+		)
+		(property "Value" "TestPoint"
+			(at 130.81 69.0879 0)
+			(hide yes)
+			(show_name no)
+			(do_not_autoplace no)
+			(effects
+				(font
+					(size 1.27 1.27)
+				)
+				(justify left)
+			)
+		)
+		(property "Footprint" "Connector_PinHeader_2.00mm:PinHeader_1x01_P2.00mm_Vertical"
+			(at 133.35 71.12 0)
+			(hide yes)
+			(show_name no)
+			(do_not_autoplace no)
+			(effects
+				(font
+					(size 1.27 1.27)
+				)
+			)
+		)
+		(property "Datasheet" ""
+			(at 133.35 71.12 0)
+			(hide yes)
+			(show_name no)
+			(do_not_autoplace no)
+			(effects
+				(font
+					(size 1.27 1.27)
+				)
+			)
+		)
+		(property "Description" "test point"
+			(at 128.27 71.12 0)
+			(hide yes)
+			(show_name no)
+			(do_not_autoplace no)
+			(effects
+				(font
+					(size 1.27 1.27)
+				)
+			)
+		)
+		(pin "1"
+		)
+		(instances
+			(project "bj-magistrska"
+				(path "/6822ed0d-de6e-44f8-850c-f571d41ba3a1/db2bed50-6fec-42f4-bd2a-90f8a985e97f"
+					(reference "TP15")
+					(unit 1)
+				)
+			)
+		)
+	)
+	(symbol
 		(lib_id "PCM_Amplifier_Operational_AKL:TSV732IS")
 		(at 250.19 213.36 0)
@@
 			)
 		)
-		(property "Value" "1k"
+		(property "Value" "100R"
 			(at 95.25 156.21 90)
 			(show_name no)

Commit message: Done some work on the PCB. Will rip it up to see if there is a better wway to run current of the coil.
Parts:
- removed C10: 1n5, PCM_Capacitor_SMD_AKL:C_0603_1608Metric, symbol PCM_Capacitor_AKL:C_0603
- removed C6: 22n, PCM_Capacitor_SMD_AKL:C_0603_1608Metric, symbol PCM_Capacitor_AKL:C_0603
- removed C8, C9: 100n, PCM_Capacitor_SMD_AKL:C_0603_1608Metric, symbol PCM_Capacitor_AKL:C_0603
- removed NT1: NetTie_2, NetTie:NetTie-2_THT_Pad0.3mm, symbol Device:NetTie_2
- removed R14: 100R, PCM_Resistor_SMD_AKL:R_0603_1608Metric, symbol PCM_Resistor_AKL:R_0603
- removed R15, R19: 100k, PCM_Resistor_SMD_AKL:R_0603_1608Metric, symbol PCM_Resistor_AKL:R_0603
- removed R16: 180k, PCM_Resistor_SMD_AKL:R_0603_1608Metric, symbol PCM_Resistor_AKL:R_0603
- removed R17: 1k8, PCM_Resistor_SMD_AKL:R_0603_1608Metric, symbol PCM_Resistor_AKL:R_0603
- removed R18: 220R, PCM_Resistor_SMD_AKL:R_0603_1608Metric, symbol PCM_Resistor_AKL:R_0603
- removed TP15, TP6, TP7: TestPoint, Connector_PinHeader_2.00mm:PinHeader_1x01_P2.00mm_Vertical, symbol Connector:TestPoint
- removed U3: TSV732IS, PCM_Package_SO_AKL:MSOP-8_3x3mm_P0.65mm, symbol PCM_Amplifier_Operational_AKL:TSV732IS
- added C28: 100n, PCM_Capacitor_SMD_AKL:C_0603_1608Metric, symbol PCM_Capacitor_AKL:C_0603
- added U11: INA240A2D, Package_SO:SOIC-8_3.9x4.9mm_P1.27mm, symbol Amplifier_Current:INA240A2D
Connections:
- net GNDPWR is gone; now on net GND: R9.2
- net +5VA: now also C28.1, U11.6 (V+)
- net GND: now also C28.2, U11.1 (-), U11.2 (GND), U11.3 (REF2), U11.4 (GND), U11.7 (REF1)
- net at C21.2, Q1.S, R9.1: now also U11.8 (+)
- net at R20.1: now also U11.5
Other:
- moved on the sheet: C11, R20, R9, TP3
